Commit message: modifying waffle model

File: turtlebot3_custom_description/urdf/turtlebot3_burger.urdf.xacro (robot description, xacro)
@@ -4,5 +4,5 @@
   <xacro:include filename="$(find turtlebot3_custom_description)/urdf/common_properties.xacro"/>
   <xacro:include filename="$(find turtlebot3_custom_description)/urdf/turtlebot3_burger.gazebo.xacro"/>
-  <burger_sensor_macro prefix="burger1"/>
+  <burger_sensor_macro prefix="$(arg robot_namespace)"/>
   <link name="$(arg robot_namespace)_base_footprint"/>
   <joint name="$(arg robot_namespace)_base_joint" type="fixed">

File: turtlebot3_custom_description/urdf/turtlebot3_waffle.gazebo.xacro (robot description, xacro)
@@ -4,176 +4,178 @@
   <xacro:arg name="camera_visual" default="false"/>
   <xacro:arg name="imu_visual"    default="false"/>
-  <gazebo reference="base_link">
-    <material>Gazebo/DarkGrey</material>
-  </gazebo>
-  <gazebo reference="wheel_left_link">
-    <mu1>0.1</mu1>
-    <mu2>0.1</mu2>
-    <kp>500000.0</kp>
-    <kd>10.0</kd>
-    <minDepth>0.001</minDepth>
-    <maxVel>0.1</maxVel>
-    <fdir1>1 0 0</fdir1>
-    <material>Gazebo/FlatBlack</material>
-  </gazebo>
-  <gazebo reference="wheel_right_link">
-    <mu1>0.1</mu1>
-    <mu2>0.1</mu2>
-    <kp>500000.0</kp>
-    <kd>10.0</kd>
-    <minDepth>0.001</minDepth>
-    <maxVel>0.1</maxVel>
-    <fdir1>1 0 0</fdir1>
-    <material>Gazebo/FlatBlack</material>
-  </gazebo>
-  <gazebo reference="caster_back_right_link">
-    <mu1>0.1</mu1>
-    <mu2>0.1</mu2>
-    <kp>1000000.0</kp>
-    <kd>100.0</kd>
-    <minDepth>0.001</minDepth>
-    <maxVel>1.0</maxVel>
-    <material>Gazebo/FlatBlack</material>
-  </gazebo>
-  <gazebo reference="caster_back_left_link">
-    <mu1>0.1</mu1>
-    <mu2>0.1</mu2>
-    <kp>1000000.0</kp>
-    <kd>100.0</kd>
-    <minDepth>0.001</minDepth>
-    <maxVel>1.0</maxVel>
-    <material>Gazebo/FlatBlack</material>
-  </gazebo>
-  <gazebo reference="imu_link">
-    <sensor type="imu" name="imu">
-      <always_on>true</always_on>
-      <visualize>$(arg imu_visual)</visualize>
-    </sensor>
-    <material>Gazebo/Grey</material>
-  </gazebo>
-  <gazebo>
-    <plugin name="turtlebot3_waffle_controller" filename="libgazebo_ros_diff_drive.so">
-      <commandTopic>cmd_vel</commandTopic>
-      <odometryTopic>odom</odometryTopic>
-      <odometryFrame>odom</odometryFrame>
-      <odometrySource>world</odometrySource>
-      <publishOdomTF>true</publishOdomTF>
-      <robotBaseFrame>base_footprint</robotBaseFrame>
-      <publishWheelTF>false</publishWheelTF>
-      <publishTf>true</publishTf>
-      <publishWheelJointState>true</publishWheelJointState>
-      <legacyMode>false</legacyMode>
-      <updateRate>30</updateRate>
-      <leftJoint>wheel_left_joint</leftJoint>
-      <rightJoint>wheel_right_joint</rightJoint>
-      <wheelSeparation>0.287</wheelSeparation>
-      <wheelDiameter>0.066</wheelDiameter>
-      <wheelAcceleration>1</wheelAcceleration>
-      <wheelTorque>10</wheelTorque>
-      <rosDebugLevel>na</rosDebugLevel>
-    </plugin>
-  </gazebo>
-  <gazebo>
-    <plugin name="imu_plugin" filename="libgazebo_ros_imu.so">
-      <alwaysOn>true</alwaysOn>
-      <bodyName>imu_link</bodyName>
-      <frameName>imu_link</frameName>
-      <topicName>imu</topicName>
-      <serviceName>imu_service</serviceName>
-      <gaussianNoise>0.0</gaussianNoise>
-      <updateRate>0</updateRate>
-      <imu>
-        <noise>
-          <type>gaussian</type>
-          <rate>
-            <mean>0.0</mean>
-            <stddev>2e-4</stddev>
-            <bias_mean>0.0000075</bias_mean>
-            <bias_stddev>0.0000008</bias_stddev>
-          </rate>
-          <accel>
-            <mean>0.0</mean>
-            <stddev>1.7e-2</stddev>
-            <bias_mean>0.1</bias_mean>
-            <bias_stddev>0.001</bias_stddev>
-          </accel>
-        </noise>
-      </imu>
-    </plugin>
-  </gazebo>
-  <gazebo reference="base_scan">
-    <material>Gazebo/FlatBlack</material>
-    <sensor type="ray" name="lds_lfcd_sensor">
-      <pose>0 0 0 0 0 0</pose>
-      <visualize>$(arg laser_visual)</visualize>
-      <update_rate>5</update_rate>
-      <ray>
-        <scan>
-          <horizontal>
-            <samples>360</samples>
-            <resolution>1</resolution>
-            <min_angle>0.0</min_angle>
-            <max_angle>6.28319</max_angle>
-          </horizontal>
-        </scan>
-        <range>
-          <min>0.120</min>
-          <max>3.5</max>
-          <resolution>0.015</resolution>
-        </range>
-        <noise>
-          <type>gaussian</type>
-          <mean>0.0</mean>
-          <stddev>0.01</stddev>
-        </noise>
-      </ray>
-      <plugin name="gazebo_ros_lds_lfcd_controller" filename="libgazebo_ros_laser.so">
-        <topicName>scan</topicName>
-        <frameName>base_scan</frameName>
+  <xacro:macro  name="waffle_sensor_macro" params="prefix">
+	<gazebo reference="${prefix}_base_link">
+      <material>Gazebo/DarkGrey</material>
+	</gazebo>
+	<gazebo reference="${prefix}_wheel_left_link">
+      <mu1>0.1</mu1>
+      <mu2>0.1</mu2>
+      <kp>500000.0</kp>
+      <kd>10.0</kd>
+      <minDepth>0.001</minDepth>
+      <maxVel>0.1</maxVel>
+      <fdir1>1 0 0</fdir1>
+      <material>Gazebo/FlatBlack</material>
+	</gazebo>
+	<gazebo reference="${prefix}_wheel_right_link">
+      <mu1>0.1</mu1>
+      <mu2>0.1</mu2>
+      <kp>500000.0</kp>
+      <kd>10.0</kd>
+      <minDepth>0.001</minDepth>
+      <maxVel>0.1</maxVel>
+      <fdir1>1 0 0</fdir1>
+      <material>Gazebo/FlatBlack</material>
+	</gazebo>
+	<gazebo reference="${prefix}_caster_back_right_link">
+      <mu1>0.1</mu1>
+      <mu2>0.1</mu2>
+      <kp>1000000.0</kp>
+      <kd>100.0</kd>
+      <minDepth>0.001</minDepth>
+      <maxVel>1.0</maxVel>
+      <material>Gazebo/FlatBlack</material>
+	</gazebo>
+	<gazebo reference="${prefix}_caster_back_left_link">
+      <mu1>0.1</mu1>
+      <mu2>0.1</mu2>
+      <kp>1000000.0</kp>
+      <kd>100.0</kd>
+      <minDepth>0.001</minDepth>
+      <maxVel>1.0</maxVel>
+      <material>Gazebo/FlatBlack</material>
+	</gazebo>
+	<gazebo reference="${prefix}_imu_link">
+      <sensor type="imu" name="imu">
+		<always_on>true</always_on>
+		<visualize>$(arg imu_visual)</visualize>
+      </sensor>
+      <material>Gazebo/Grey</material>
+	</gazebo>
+	<gazebo>
+      <plugin name="turtlebot3_waffle_controller" filename="libgazebo_ros_diff_drive.so">
+		<commandTopic>${prefix}/cmd_vel</commandTopic>
+		<odometryTopic>${prefix}/odom</odometryTopic>
+		<odometryFrame>${prefix}/odom</odometryFrame>
+		<odometrySource>world</odometrySource>
+		<publishOdomTF>true</publishOdomTF>
+		<robotBaseFrame>${prefix}_base_footprint</robotBaseFrame>
+		<publishWheelTF>false</publishWheelTF>
+		<publishTf>true</publishTf>
+		<publishWheelJointState>true</publishWheelJointState>
+		<legacyMode>false</legacyMode>
+		<updateRate>30</updateRate>
+		<leftJoint>${prefix}_wheel_left_joint</leftJoint>
+		<rightJoint>${prefix}_wheel_right_joint</rightJoint>
+		<wheelSeparation>0.287</wheelSeparation>
+		<wheelDiameter>0.066</wheelDiameter>
+		<wheelAcceleration>1</wheelAcceleration>
+		<wheelTorque>10</wheelTorque>
+		<rosDebugLevel>na</rosDebugLevel>
       </plugin>
-    </sensor>
-  </gazebo>
-  <gazebo reference="camera_rgb_frame">
-    <sensor type="depth" name="realsense_R200">
-      <always_on>true</always_on>
-      <visualize>$(arg camera_visual)</visualize>
-      <camera>
+	</gazebo>
+	<gazebo>
+      <plugin name="imu_plugin" filename="libgazebo_ros_imu.so">
+		<alwaysOn>true</alwaysOn>
+		<bodyName>${prefix}_imu_link</bodyName>
+		<frameName>${prefix}_imu_link</frameName>
+		<topicName>${prefix}/imu</topicName>
+		<serviceName>${prefix}/imu_service</serviceName>
+		<gaussianNoise>0.0</gaussianNoise>
+		<updateRate>0</updateRate>
+		<imu>
+          <noise>
+			<type>gaussian</type>
+			<rate>
+              <mean>0.0</mean>
+              <stddev>2e-4</stddev>
+              <bias_mean>0.0000075</bias_mean>
+              <bias_stddev>0.0000008</bias_stddev>
+			</rate>
+			<accel>
+              <mean>0.0</mean>
+              <stddev>1.7e-2</stddev>
+              <bias_mean>0.1</bias_mean>
+              <bias_stddev>0.001</bias_stddev>
+			</accel>
+          </noise>
+		</imu>
+      </plugin>
+	</gazebo>
+	<gazebo reference="${prefix}_base_scan">
+      <material>Gazebo/FlatBlack</material>
+      <sensor type="ray" name="lds_lfcd_sensor">
+		<pose>0 0 0 0 0 0</pose>
+		<visualize>$(arg laser_visual)</visualize>
+		<update_rate>5</update_rate>
+		<ray>
+          <scan>
+			<horizontal>
+              <samples>360</samples>
+              <resolution>1</resolution>
+              <min_angle>0.0</min_angle>
+              <max_angle>6.28319</max_angle>
+			</horizontal>
+          </scan>
+          <range>
+			<min>0.120</min>
+			<max>3.5</max>
+			<resolution>0.015</resolution>
+          </range>
+          <noise>
+			<type>gaussian</type>
+			<mean>0.0</mean>
+			<stddev>0.01</stddev>
+          </noise>
+		</ray>
+		<plugin name="gazebo_ros_lds_lfcd_controller" filename="libgazebo_ros_laser.so">
+          <topicName>${prefix}/scan</topicName>
+          <frameName>${prefix}_base_scan</frameName>
+		</plugin>
+      </sensor>
+	</gazebo>
+	<gazebo reference="${prefix}_camera_rgb_frame">
+      <sensor type="depth" name="realsense_R200">
+		<always_on>true</always_on>
+		<visualize>$(arg camera_visual)</visualize>
+		<camera>
           <horizontal_fov>1.3439</horizontal_fov>
           <image>
-              <width>1920</width>
-              <height>1080</height>
-              <format>R8G8B8</format>
+            <width>1920</width>
+            <height>1080</height>
+            <format>R8G8B8</format>
           </image>
           <depth_camera></depth_camera>
           <clip>
-              <near>0.03</near>
-              <far>100</far>
+            <near>0.03</near>
+            <far>100</far>
           </clip>
-      </camera>
-      <plugin name="camera_controller" filename="libgazebo_ros_openni_kinect.so">
-        <baseline>0.2</baseline>
-        <alwaysOn>true</alwaysOn>
-        <updateRate>30.0</updateRate>
-        <cameraName>camera</cameraName>
-        <frameName>camera_rgb_optical_frame</frameName>
-        <imageTopicName>rgb/image_raw</imageTopicName>
-        <depthImageTopicName>depth/image_raw</depthImageTopicName>
-        <pointCloudTopicName>depth/points</pointCloudTopicName>
-        <cameraInfoTopicName>rgb/camera_info</cameraInfoTopicName>
-        <depthImageCameraInfoTopicName>depth/camera_info</depthImageCameraInfoTopicName>
-        <pointCloudCutoff>0.4</pointCloudCutoff>
-            <hackBaseline>0.07</hackBaseline>
-            <distortionK1>0.0</distortionK1>
-            <distortionK2>0.0</distortionK2>
-            <distortionK3>0.0</distortionK3>
-            <distortionT1>0.0</distortionT1>
-            <distortionT2>0.0</distortionT2>
-        <CxPrime>0.0</CxPrime>
-        <Cx>0.0</Cx>
-        <Cy>0.0</Cy>
-        <focalLength>0</focalLength>
-        <hackBaseline>0</hackBaseline>
-      </plugin>
-    </sensor>
-  </gazebo>
+		</camera>
+		<plugin name="camera_controller" filename="libgazebo_ros_openni_kinect.so">
+          <baseline>0.2</baseline>
+          <alwaysOn>true</alwaysOn>
+          <updateRate>30.0</updateRate>
+          <cameraName>${prefix}/camera</cameraName>
+          <frameName>${prefix}_camera_rgb_optical_frame</frameName>
+          <imageTopicName>${prefix}/rgb/image_raw</imageTopicName>
+          <depthImageTopicName>${prefix}/depth/image_raw</depthImageTopicName>
+          <pointCloudTopicName>${prefix}/depth/points</pointCloudTopicName>
+          <cameraInfoTopicName>${prefix}/rgb/camera_info</cameraInfoTopicName>
+          <depthImageCameraInfoTopicName>${prefix}/depth/camera_info</depthImageCameraInfoTopicName>
+          <pointCloudCutoff>0.4</pointCloudCutoff>
+          <hackBaseline>0.07</hackBaseline>
+          <distortionK1>0.0</distortionK1>
+          <distortionK2>0.0</distortionK2>
+          <distortionK3>0.0</distortionK3>
+          <distortionT1>0.0</distortionT1>
+          <distortionT2>0.0</distortionT2>
+          <CxPrime>0.0</CxPrime>
+          <Cx>0.0</Cx>
+          <Cy>0.0</Cy>
+          <focalLength>0</focalLength>
+          <hackBaseline>0</hackBaseline>
+		</plugin>
+      </sensor>
+	</gazebo>
+  </xacro:macro>
 </robot>

File: turtlebot3_custom_description/urdf/turtlebot3_waffle.urdf.xacro (robot description, xacro)
@@ -1,21 +1,23 @@
 <?xml version="1.0" ?>
 <robot name="turtlebot3_waffle" xmlns:xacro="http://ros.org/wiki/xacro">
-  <xacro:include filename="$(find turtlebot3_description)/urdf/common_properties.xacro"/>
-  <xacro:include filename="$(find turtlebot3_description)/urdf/turtlebot3_waffle.gazebo.xacro"/>
+  <xacro:arg name="robot_namespace" default="waffle1"/>
+  <xacro:include filename="$(find turtlebot3_custom_description)/urdf/common_properties.xacro"/>
+  <xacro:include filename="$(find turtlebot3_custom_description)/urdf/turtlebot3_waffle.gazebo.xacro"/>
+  <waffle_sensor_macro prefix="$(arg robot_namespace)"/>
   <xacro:property name="r200_cam_rgb_px" value="0.005"/>
   <xacro:property name="r200_cam_rgb_py" value="0.018"/>
   <xacro:property name="r200_cam_rgb_pz" value="0.013"/>
   <xacro:property name="r200_cam_depth_offset" value="0.01"/>
-  <link name="base_footprint"/>
-  <joint name="base_joint" type="fixed">
-    <parent link="base_footprint"/>
-    <child link="base_link" />
+  <link name="$(arg robot_namespace)_base_footprint"/>
+  <joint name="$(arg robot_namespace)_base_joint" type="fixed">
+    <parent link="$(arg robot_namespace)_base_footprint"/>
+    <child link="$(arg robot_namespace)_base_link" />
     <origin xyz="0 0 0.010" rpy="0 0 0"/>
   </joint>
-  <link name="base_link">
+  <link name="$(arg robot_namespace)_base_link">
     <visual>
       <origin xyz="-0.064 0 0.0" rpy="0 0 0"/>
       <geometry>
-        <mesh filename="package://turtlebot3_description/meshes/bases/waffle_base.stl" scale="0.001 0.001 0.001"/>
+        <mesh filename="package://turtlebot3_custom_description/meshes/bases/waffle_base.stl" scale="0.001 0.001 0.001"/>
       </geometry>
       <material name="light_black"/>
@@ -35,15 +37,15 @@
     </inertial>
   </link>
-  <joint name="wheel_left_joint" type="continuous">
-    <parent link="base_link"/>
-    <child link="wheel_left_link"/>
+  <joint name="$(arg robot_namespace)_wheel_left_joint" type="continuous">
+    <parent link="$(arg robot_namespace)_base_link"/>
+    <child link="$(arg robot_namespace)_wheel_left_link"/>
     <origin xyz="0.0 0.144 0.023" rpy="-1.57 0 0"/>
     <axis xyz="0 0 1"/>
   </joint>
-  <link name="wheel_left_link">
+  <link name="$(arg robot_namespace)_wheel_left_link">
     <visual>
       <origin xyz="0 0 0" rpy="1.57 0 0"/>
       <geometry>
-        <mesh filename="package://turtlebot3_description/meshes/wheels/left_tire.stl" scale="0.001 0.001 0.001"/>
+        <mesh filename="package://turtlebot3_custom_description/meshes/wheels/left_tire.stl" scale="0.001 0.001 0.001"/>
       </geometry>
       <material name="dark"/>
@@ -63,15 +65,15 @@
       </inertial>
   </link>
-  <joint name="wheel_right_joint" type="continuous">
-    <parent link="base_link"/>
-    <child link="wheel_right_link"/>
+  <joint name="$(arg robot_namespace)_wheel_right_joint" type="continuous">
+    <parent link="$(arg robot_namespace)_base_link"/>
+    <child link="$(arg robot_namespace)_wheel_right_link"/>
     <origin xyz="0.0 -0.144 0.023" rpy="-1.57 0 0"/>
     <axis xyz="0 0 1"/>
   </joint>
-  <link name="wheel_right_link">
+  <link name="$(arg robot_namespace)_wheel_right_link">
     <visual>
       <origin xyz="0 0 0" rpy="1.57 0 0"/>
       <geometry>
-        <mesh filename="package://turtlebot3_description/meshes/wheels/right_tire.stl" scale="0.001 0.001 0.001"/>
+        <mesh filename="package://turtlebot3_custom_description/meshes/wheels/right_tire.stl" scale="0.001 0.001 0.001"/>
       </geometry>
       <material name="dark"/>
@@ -91,10 +93,10 @@
       </inertial>
   </link>
-  <joint name="caster_back_right_joint" type="fixed">
-    <parent link="base_link"/>
-    <child link="caster_back_right_link"/>
+  <joint name="$(arg robot_namespace)_caster_back_right_joint" type="fixed">
+    <parent link="$(arg robot_namespace)_base_link"/>
+    <child link="$(arg robot_namespace)_caster_back_right_link"/>
     <origin xyz="-0.177 -0.064 -0.004" rpy="-1.57 0 0"/>
   </joint>
-  <link name="caster_back_right_link">
+  <link name="$(arg robot_namespace)_caster_back_right_link">
     <collision>
       <origin xyz="0 0.001 0" rpy="0 0 0"/>
@@ -111,10 +113,10 @@
     </inertial>
   </link>
-  <joint name="caster_back_left_joint" type="fixed">
-    <parent link="base_link"/>
-    <child link="caster_back_left_link"/>
+  <joint name="$(arg robot_namespace)_caster_back_left_joint" type="fixed">
+    <parent link="$(arg robot_namespace)_base_link"/>
+    <child link="$(arg robot_namespace)_caster_back_left_link"/>
     <origin xyz="-0.177 0.064 -0.004" rpy="-1.57 0 0"/>
   </joint>
-  <link name="caster_back_left_link">
+  <link name="$(arg robot_namespace)_caster_back_left_link">
     <collision>
       <origin xyz="0 0.001 0" rpy="0 0 0"/>
@@ -131,20 +133,20 @@
     </inertial>
   </link>
-  <joint name="imu_joint" type="fixed">
-    <parent link="base_link"/>
-    <child link="imu_link"/>
+  <joint name="$(arg robot_namespace)_imu_joint" type="fixed">
+    <parent link="$(arg robot_namespace)_base_link"/>
+    <child link="$(arg robot_namespace)_imu_link"/>
     <origin xyz="0.0 0 0.068" rpy="0 0 0"/>
   </joint>
-  <link name="imu_link"/>
-  <joint name="scan_joint" type="fixed">
-    <parent link="base_link"/>
-    <child link="base_scan"/>
+  <link name="$(arg robot_namespace)_imu_link"/>
+  <joint name="$(arg robot_namespace)_scan_joint" type="fixed">
+    <parent link="$(arg robot_namespace)_base_link"/>
+    <child link="$(arg robot_namespace)_base_scan"/>
     <origin xyz="-0.064 0 0.122" rpy="0 0 0"/>
   </joint>
-  <link name="base_scan">
-    <visual>
-      <origin xyz="0 0 0" rpy="0 0 0"/>
-      <geometry>
-        <mesh filename="package://turtlebot3_description/meshes/sensors/lds.stl" scale="0.001 0.001 0.001"/>
+  <link name="$(arg robot_namespace)_base_scan">
+    <visual>
+      <origin xyz="0 0 0" rpy="0 0 0"/>
+      <geometry>
+        <mesh filename="package://turtlebot3_custom_description/meshes/sensors/lds.stl" scale="0.001 0.001 0.001"/>
       </geometry>
       <material name="dark"/>
@@ -164,14 +166,14 @@
     </inertial>
   </link>
-  <joint name="camera_joint" type="fixed">
+  <joint name="$(arg robot_namespace)_camera_joint" type="fixed">
     <origin xyz="0.064 -0.065 0.094" rpy="0 0 0"/>
-    <parent link="base_link"/>
-    <child link="camera_link"/>
-  </joint>
-  <link name="camera_link">
+    <parent link="$(arg robot_namespace)_base_link"/>
+    <child link="$(arg robot_namespace)_camera_link"/>
+  </joint>
+  <link name="$(arg robot_namespace)_camera_link">
     <visual>
      <origin xyz="0 0 0" rpy="1.57 0 1.57"/>
       <geometry>
-       <mesh filename="package://turtlebot3_description/meshes/sensors/r200.dae" />
+       <mesh filename="package://turtlebot3_custom_description/meshes/sensors/r200.dae" />
       </geometry>
     </visual>
@@ -191,27 +193,27 @@
     </inertial>-->
   </link>
-  <joint name="camera_rgb_joint" type="fixed">
+  <joint name="$(arg robot_namespace)_camera_rgb_joint" type="fixed">
     <origin xyz="${r200_cam_rgb_px} ${r200_cam_rgb_py} ${r200_cam_rgb_pz}" rpy="0 0 0"/>
-    <parent link="camera_link"/>
-    <child link="camera_rgb_frame"/>
-  </joint>
-  <link name="camera_rgb_frame"/>
-  <joint name="camera_rgb_optical_joint" type="fixed">
+    <parent link="$(arg robot_namespace)_camera_link"/>
+    <child link="$(arg robot_namespace)_camera_rgb_frame"/>
+  </joint>
+  <link name="$(arg robot_namespace)_camera_rgb_frame"/>
+  <joint name="$(arg robot_namespace)_camera_rgb_optical_joint" type="fixed">
     <origin xyz="0 0 0" rpy="-1.57 0 -1.57"/>
-    <parent link="camera_rgb_frame"/>
-    <child link="camera_rgb_optical_frame"/>
-  </joint>
-  <link name="camera_rgb_optical_frame"/>
-  <joint name="camera_depth_joint" type="fixed">
+    <parent link="$(arg robot_namespace)_camera_rgb_frame"/>
+    <child link="$(arg robot_namespace)_camera_rgb_optical_frame"/>
+  </joint>
+  <link name="$(arg robot_namespace)_camera_rgb_optical_frame"/>
+  <joint name="$(arg robot_namespace)_camera_depth_joint" type="fixed">
     <origin xyz="${r200_cam_rgb_px} ${r200_cam_rgb_py + r200_cam_depth_offset} ${r200_cam_rgb_pz}" rpy="0 0 0"/>
-    <parent link="camera_link"/>
-    <child link="camera_depth_frame"/>
-  </joint>
-  <link name="camera_depth_frame"/>
-  <joint name="camera_depth_optical_joint" type="fixed">
+    <parent link="$(arg robot_namespace)_camera_link"/>
+    <child link="$(arg robot_namespace)_camera_depth_frame"/>
+  </joint>
+  <link name="$(arg robot_namespace)_camera_depth_frame"/>
+  <joint name="$(arg robot_namespace)_camera_depth_optical_joint" type="fixed">
     <origin xyz="0 0 0" rpy="-1.57 0 -1.57"/>
-    <parent link="camera_depth_frame"/>
-    <child link="camera_depth_optical_frame"/>
-  </joint>
-  <link name="camera_depth_optical_frame"/>
+    <parent link="$(arg robot_namespace)_camera_depth_frame"/>
+    <child link="$(arg robot_namespace)_camera_depth_optical_frame"/>
+  </joint>
+  <link name="$(arg robot_namespace)_camera_depth_optical_frame"/>
 </robot>
