Commit message: migrated burger to ros2 galactic. TODO: (1) desc for how to pass arguments to launch (2) migrate waffle and waffle_pi (3) prepare each sim_{model}.rviz
Signed-off-by: soblin <hilo.soblin@gmail.com>

File: turtlebot3_custom_description/urdf/common_properties.xacro (robot description, xacro)
@@ -3,5 +3,5 @@
   <!-- Init colour -->
   <material name="black">
-      <color rgba="0.0 0.0 0.0 1.0"/>
+    <color rgba="0.0 0.0 0.0 1.0"/>
   </material>
   <material name="dark">

File: turtlebot3_custom_description/urdf/turtlebot3_burger.gazebo.xacro (robot description, xacro)
@@ -12,6 +12,6 @@
       <kp>500000.0</kp>
       <kd>10.0</kd>
-      <minDepth>0.001</minDepth>
-      <maxVel>0.1</maxVel>
+      <min_depth>0.001</min_depth>
+      <max_vel>0.1</max_vel>
       <fdir1>1 0 0</fdir1>
       <material>Gazebo/FlatBlack</material>
@@ -22,6 +22,6 @@
       <kp>500000.0</kp>
       <kd>10.0</kd>
-      <minDepth>0.001</minDepth>
-      <maxVel>0.1</maxVel>
+      <min_depth>0.001</min_depth>
+      <max_vel>0.1</max_vel>
       <fdir1>1 0 0</fdir1>
       <material>Gazebo/FlatBlack</material>
@@ -32,6 +32,6 @@
       <kp>1000000.0</kp>
       <kd>100.0</kd>
-      <minDepth>0.001</minDepth>
-      <maxVel>1.0</maxVel>
+      <min_depth>0.001</min_depth>
+      <max_vel>1.0</max_vel>
       <material>Gazebo/FlatBlack</material>
 	</gazebo>
@@ -45,84 +45,96 @@
 	<gazebo>
       <plugin name="turtlebot3_burger_controller" filename="libgazebo_ros_diff_drive.so">
-		<commandTopic>${prefix}_cmd_vel</commandTopic>
-		<odometryTopic>${prefix}_odom</odometryTopic>
-		<odometryFrame>${prefix}_odom</odometryFrame>
-		<odometrySource>world</odometrySource>
-		<publishOdomTF>true</publishOdomTF>
-		<robotBaseFrame>${prefix}_base_footprint</robotBaseFrame>
-		<publishWheelTF>false</publishWheelTF>
-		<publishTf>true</publishTf>
-		<publishWheelJointState>true</publishWheelJointState>
-		<legacyMode>false</legacyMode>
-		<updateRate>30</updateRate>
-		<leftJoint>${prefix}_wheel_left_joint</leftJoint>
-		<rightJoint>${prefix}_wheel_right_joint</rightJoint>
-		<wheelSeparation>0.160</wheelSeparation>
-		<wheelDiameter>0.066</wheelDiameter>
-		<wheelAcceleration>1</wheelAcceleration>
-		<wheelTorque>10</wheelTorque>
-		<rosDebugLevel>na</rosDebugLevel>
+		<update_rate>30</update_rate>
+		<left_joint>${prefix}_wheel_left_joint</left_joint>
+		<right_joint>${prefix}_wheel_right_joint</right_joint>
+		<wheel_separation>0.160</wheel_separation>
+		<wheel_diameter>0.066</wheel_diameter>
+		<max_wheel_torque>20</max_wheel_torque>
+		<max_wheel_acceleration>1.0</max_wheel_acceleration>
+		<publish_odom>true</publish_odom>
+		<publish_odom_tf>true</publish_odom_tf>
+		<publish_wheel_tf>false</publish_wheel_tf>
+		<odometry_frame>${prefix}_odom</odometry_frame>
+		<robot_base_frame>${prefix}_base_footprint</robot_base_frame>
+		<!-- https://github.com/ros-simulation/gazebo_ros_pkgs/wiki/ROS-2-Migration:-Diff-drive -->
+		<ros>
+		  <remapping>cmd_vel:=${prefix}_cmd_vel</remapping>
+		  <remapping>odom:=${prefix}_odom</remapping>
+		</ros>
       </plugin>
 	</gazebo>
-	<gazebo>
-      <plugin name="imu_plugin" filename="libgazebo_ros_imu.so">
-		<alwaysOn>true</alwaysOn>
-		<bodyName>${prefix}_imu_link</bodyName>
-		<frameName>${prefix}_imu_link</frameName>
-		<topicName>${prefix}_imu</topicName>
-		<serviceName>${prefix}_imu_service</serviceName>
-		<gaussianNoise>0.0</gaussianNoise>
-		<updateRate>0</updateRate>
+	<!--gazebo>
+		<plugin name="imu_plugin" filename="libgazebo_ros_imu.so">
+		<always_on>true</always_on>
+		<body_name>${prefix}_imu_link</body_name>
+		<frame_name>${prefix}_imu_link</frame_name>
+		<topic_name>${prefix}_imu</topic_name>
+		<service_name>${prefix}_imu_service</service_name>
+		<gaussian_noise>0.0</gaussian_noise>
+		<update_rate>0</update_rate>
 		<imu>
-          <noise>
-			<type>gaussian</type>
-			<rate>
-              <mean>0.0</mean>
-              <stddev>2e-4</stddev>
-              <bias_mean>0.0000075</bias_mean>
-              <bias_stddev>0.0000008</bias_stddev>
-			</rate>
-			<accel>
-              <mean>0.0</mean>
-              <stddev>1.7e-2</stddev>
-              <bias_mean>0.1</bias_mean>
-              <bias_stddev>0.001</bias_stddev>
-			</accel>
-          </noise>
+        <noise>
+		<type>gaussian</type>
+		<rate>
+        <mean>0.0</mean>
+        <stddev>2e-4</stddev>
+        <bias_mean>0.0000075</bias_mean>
+        <bias_stddev>0.0000008</bias_stddev>
+		</rate>
+		<accel>
+        <mean>0.0</mean>
+        <stddev>1.7e-2</stddev>
+        <bias_mean>0.1</bias_mean>
+        <bias_stddev>0.001</bias_stddev>
+		</accel>
+        </noise>
 		</imu>
-      </plugin>
-	</gazebo>
+		</plugin>
+		</gazebo-->
 	<gazebo reference="${prefix}_base_scan">
-      <material>Gazebo/FlatBlack</material>
       <sensor type="ray" name="lds_lfcd_sensor">
-		<pose>0 0 0 0 0 0</pose>
-		<visualize>$(arg laser_visual)</visualize>
-		<update_rate>5</update_rate>
-		<ray>
+        <always_on>true</always_on>
+        <visualize>true</visualize>
+        <pose>-0.032 0 0.171 0 0 0</pose>
+        <update_rate>5</update_rate>
+        <ray>
           <scan>
-			<horizontal>
+            <horizontal>
               <samples>360</samples>
-              <resolution>1</resolution>
-              <min_angle>0.0</min_angle>
-              <max_angle>6.28319</max_angle>
-			</horizontal>
+              <resolution>1.000000</resolution>
+              <min_angle>0.000000</min_angle>
+              <max_angle>6.280000</max_angle>
+            </horizontal>
           </scan>
           <range>
-			<min>0.120</min>
-			<max>3.5</max>
-			<resolution>0.015</resolution>
+            <min>0.120000</min>
+            <max>3.5</max>
+            <resolution>0.015000</resolution>
           </range>
           <noise>
-			<type>gaussian</type>
-			<mean>0.0</mean>
-			<stddev>0.01</stddev>
+            <type>gaussian</type>
+            <mean>0.0</mean>
+            <stddev>0.01</stddev>
           </noise>
-		</ray>
-		<plugin name="gazebo_ros_lds_lfcd_controller" filename="libgazebo_ros_laser.so">
-          <topicName>${prefix}_scan</topicName>
-          <frameName>${prefix}_base_scan</frameName>
+        </ray>
+		<plugin name="gazebo_ros_lds_lfcd_controller" filename="libgazebo_ros_ray_sensor.so">
+          <ros>
+            <remapping>~/out:=${prefix}_scan</remapping>
+          </ros>
+          <output_type>sensor_msgs/LaserScan</output_type>
+          <frame_name>${prefix}_base_scan</frame_name>
 		</plugin>
       </sensor>
 	</gazebo>
+	<gazebo>
+      <plugin name="turtlebot3_burger_joint_state" filename="libgazebo_ros_joint_state_publisher.so">
+		<ros>
+		  <remapping>~/out:=joint_states</remapping>
+		</ros>
+		<update_rate>30</update_rate>
+		<joint_name>${prefix}_wheel_left_joint</joint_name>
+		<joint_name>${prefix}_wheel_right_joint</joint_name>
+	  </plugin>
+	</gazebo>
   </xacro:macro>
 </robot>

File: turtlebot3_custom_description/urdf/turtlebot3_burger.urdf.xacro (robot description, xacro)
@@ -15,5 +15,5 @@
       <origin xyz="-0.032 0 0.0" rpy="0 0 0"/>
       <geometry>
-        <mesh filename="package://turtlebot3_custom_description/meshes/bases/burger_base.stl" scale="0.001 0.001 0.001"/>
+        <mesh filename="package://turtlebot3_custom_description/meshes/burger_base.dae" scale="0.001 0.001 0.001"/>
       </geometry>
       <material name="light_black"/>
@@ -43,5 +43,5 @@
       <origin xyz="0 0 0" rpy="1.57 0 0"/>
       <geometry>
-        <mesh filename="package://turtlebot3_custom_description/meshes/wheels/left_tire.stl" scale="0.001 0.001 0.001"/>
+        <mesh filename="package://turtlebot3_custom_description/meshes/tire.dae" scale="0.001 0.001 0.001"/>
       </geometry>
       <material name="dark"/>
@@ -59,5 +59,5 @@
                iyy="1.1192413e-05" iyz="-1.4400107e-11"
                izz="2.0712558e-05" />
-      </inertial>
+    </inertial>
   </link>
   <joint name="$(arg robot_namespace)_wheel_right_joint" type="continuous">
@@ -71,5 +71,5 @@
       <origin xyz="0 0 0" rpy="1.57 0 0"/>
       <geometry>
-        <mesh filename="package://turtlebot3_custom_description/meshes/wheels/right_tire.stl" scale="0.001 0.001 0.001"/>
+        <mesh filename="package://turtlebot3_custom_description/meshes/tire.dae" scale="0.001 0.001 0.001"/>
       </geometry>
       <material name="dark"/>
@@ -87,5 +87,5 @@
                iyy="1.1192413e-05" iyz="-1.4400107e-11"
                izz="2.0712558e-05" />
-      </inertial>
+    </inertial>
   </link>
   <joint name="$(arg robot_namespace)_caster_back_joint" type="fixed">
@@ -124,5 +124,5 @@
       <origin xyz="0 0 0.0" rpy="0 0 0"/>
       <geometry>
-        <mesh filename="package://turtlebot3_custom_description/meshes/sensors/lds.stl" scale="0.001 0.001 0.001"/>
+        <mesh filename="package://turtlebot3_custom_description/meshes/lds.dae" scale="0.001 0.001 0.001"/>
       </geometry>
       <material name="dark"/>

File: turtlebot3_custom_description/urdf/turtlebot3_waffle.urdf.xacro (robot description, xacro)
@@ -63,5 +63,5 @@
                iyy="1.1192413e-05" iyz="-1.4400107e-11"
                izz="2.0712558e-05" />
-      </inertial>
+    </inertial>
   </link>
   <joint name="$(arg robot_namespace)_wheel_right_joint" type="continuous">
@@ -91,5 +91,5 @@
                iyy="1.1192413e-05" iyz="-1.4400107e-11"
                izz="2.0712558e-05" />
-      </inertial>
+    </inertial>
   </link>
   <joint name="$(arg robot_namespace)_caster_back_right_joint" type="fixed">
@@ -173,7 +173,7 @@
   <link name="$(arg robot_namespace)_camera_link">
     <visual>
-     <origin xyz="0 0 0" rpy="1.57 0 1.57"/>
-      <geometry>
-       <mesh filename="package://turtlebot3_custom_description/meshes/sensors/r200.dae" />
+      <origin xyz="0 0 0" rpy="1.57 0 1.57"/>
+      <geometry>
+		<mesh filename="package://turtlebot3_custom_description/meshes/sensors/r200.dae" />
       </geometry>
     </visual>
@@ -185,11 +185,11 @@
     </collision>
     <!-- This inertial field needs doesn't contain reliable data!! -->
-<!--   <inertial>
-      <mass value="0.564" />
-      <origin xyz="0 0 0" />
-      <inertia ixx="0.003881243" ixy="0.0" ixz="0.0"
-               iyy="0.000498940" iyz="0.0"
-               izz="0.003879257" />
-    </inertial>-->
+	<!--   <inertial>
+		 <mass value="0.564" />
+		 <origin xyz="0 0 0" />
+		 <inertia ixx="0.003881243" ixy="0.0" ixz="0.0"
+         iyy="0.000498940" iyz="0.0"
+         izz="0.003879257" />
+		 </inertial>-->
   </link>
   <joint name="$(arg robot_namespace)_camera_rgb_joint" type="fixed">

File: turtlebot3_custom_description/urdf/turtlebot3_waffle_pi.urdf.xacro (robot description, xacro)
@@ -59,5 +59,5 @@
                iyy="1.1192413e-05" iyz="-1.4400107e-11"
                izz="2.0712558e-05" />
-      </inertial>
+    </inertial>
   </link>
   <joint name="$(arg robot_namespace)_wheel_right_joint" type="continuous">
@@ -87,5 +87,5 @@
                iyy="1.1192413e-05" iyz="-1.4400107e-11"
                izz="2.0712558e-05" />
-      </inertial>
+    </inertial>
   </link>
   <joint name="$(arg robot_namespace)_caster_back_right_joint" type="fixed">
