Commit message: 1) changed urdf link name from prefix/link to prefix_link 2) rename gazebo's input/output {cmd, odom, scan} to prefix/{cmd, odom, scan} TODO do the same thing for waffle, waffle_pi as well

File: turtlebot3_custom_description/urdf/turtlebot3_burger.gazebo.xacro (robot description, xacro)
@@ -3,124 +3,126 @@
   <xacro:arg name="laser_visual" default="false"/>
   <xacro:arg name="imu_visual"   default="false"/>
-  <gazebo reference="base_link">
-    <material>Gazebo/DarkGrey</material>
-  </gazebo>
-  <gazebo reference="wheel_left_link">
-    <mu1>0.1</mu1>
-    <mu2>0.1</mu2>
-    <kp>500000.0</kp>
-    <kd>10.0</kd>
-    <minDepth>0.001</minDepth>
-    <maxVel>0.1</maxVel>
-    <fdir1>1 0 0</fdir1>
-    <material>Gazebo/FlatBlack</material>
-  </gazebo>
-  <gazebo reference="wheel_right_link">
-    <mu1>0.1</mu1>
-    <mu2>0.1</mu2>
-    <kp>500000.0</kp>
-    <kd>10.0</kd>
-    <minDepth>0.001</minDepth>
-    <maxVel>0.1</maxVel>
-    <fdir1>1 0 0</fdir1>
-    <material>Gazebo/FlatBlack</material>
-  </gazebo>
-  <gazebo reference="caster_back_link">
-    <mu1>0.1</mu1>
-    <mu2>0.1</mu2>
-    <kp>1000000.0</kp>
-    <kd>100.0</kd>
-    <minDepth>0.001</minDepth>
-    <maxVel>1.0</maxVel>
-    <material>Gazebo/FlatBlack</material>
-  </gazebo>
-  <gazebo reference="imu_link">
-    <sensor type="imu" name="imu">
-      <always_on>true</always_on>
-      <visualize>$(arg imu_visual)</visualize>
-    </sensor>
-    <material>Gazebo/FlatBlack</material>
-  </gazebo>
-  <gazebo>
-    <plugin name="turtlebot3_burger_controller" filename="libgazebo_ros_diff_drive.so">
-      <commandTopic>cmd_vel</commandTopic>
-      <odometryTopic>odom</odometryTopic>
-      <odometryFrame>odom</odometryFrame>
-      <odometrySource>world</odometrySource>
-      <publishOdomTF>true</publishOdomTF>
-      <robotBaseFrame>base_footprint</robotBaseFrame>
-      <publishWheelTF>false</publishWheelTF>
-      <publishTf>true</publishTf>
-      <publishWheelJointState>true</publishWheelJointState>
-      <legacyMode>false</legacyMode>
-      <updateRate>30</updateRate>
-      <leftJoint>wheel_left_joint</leftJoint>
-      <rightJoint>wheel_right_joint</rightJoint>
-      <wheelSeparation>0.160</wheelSeparation>
-      <wheelDiameter>0.066</wheelDiameter>
-      <wheelAcceleration>1</wheelAcceleration>
-      <wheelTorque>10</wheelTorque>
-      <rosDebugLevel>na</rosDebugLevel>
-    </plugin>
-  </gazebo>
-  <gazebo>
-    <plugin name="imu_plugin" filename="libgazebo_ros_imu.so">
-      <alwaysOn>true</alwaysOn>
-      <bodyName>imu_link</bodyName>
-      <frameName>imu_link</frameName>
-      <topicName>imu</topicName>
-      <serviceName>imu_service</serviceName>
-      <gaussianNoise>0.0</gaussianNoise>
-      <updateRate>0</updateRate>
-      <imu>
-        <noise>
-          <type>gaussian</type>
-          <rate>
-            <mean>0.0</mean>
-            <stddev>2e-4</stddev>
-            <bias_mean>0.0000075</bias_mean>
-            <bias_stddev>0.0000008</bias_stddev>
-          </rate>
-          <accel>
-            <mean>0.0</mean>
-            <stddev>1.7e-2</stddev>
-            <bias_mean>0.1</bias_mean>
-            <bias_stddev>0.001</bias_stddev>
-          </accel>
-        </noise>
-      </imu>
-    </plugin>
-  </gazebo>
-  <gazebo reference="base_scan">
-    <material>Gazebo/FlatBlack</material>
-    <sensor type="ray" name="lds_lfcd_sensor">
-      <pose>0 0 0 0 0 0</pose>
-      <visualize>$(arg laser_visual)</visualize>
-      <update_rate>5</update_rate>
-      <ray>
-        <scan>
-          <horizontal>
-            <samples>360</samples>
-            <resolution>1</resolution>
-            <min_angle>0.0</min_angle>
-            <max_angle>6.28319</max_angle>
-          </horizontal>
-        </scan>
-        <range>
-          <min>0.120</min>
-          <max>3.5</max>
-          <resolution>0.015</resolution>
-        </range>
-        <noise>
-          <type>gaussian</type>
-          <mean>0.0</mean>
-          <stddev>0.01</stddev>
-        </noise>
-      </ray>
-      <plugin name="gazebo_ros_lds_lfcd_controller" filename="libgazebo_ros_laser.so">
-        <topicName>scan</topicName>
-        <frameName>base_scan</frameName>
+  <xacro:macro name="burger_sensor_macro" params="prefix">
+	<gazebo reference="${prefix}_base_link">
+      <material>Gazebo/DarkGrey</material>
+	</gazebo>
+	<gazebo reference="${prefix}_wheel_left_link">
+      <mu1>0.1</mu1>
+      <mu2>0.1</mu2>
+      <kp>500000.0</kp>
+      <kd>10.0</kd>
+      <minDepth>0.001</minDepth>
+      <maxVel>0.1</maxVel>
+      <fdir1>1 0 0</fdir1>
+      <material>Gazebo/FlatBlack</material>
+	</gazebo>
+	<gazebo reference="${prefix}_wheel_right_link">
+      <mu1>0.1</mu1>
+      <mu2>0.1</mu2>
+      <kp>500000.0</kp>
+      <kd>10.0</kd>
+      <minDepth>0.001</minDepth>
+      <maxVel>0.1</maxVel>
+      <fdir1>1 0 0</fdir1>
+      <material>Gazebo/FlatBlack</material>
+	</gazebo>
+	<gazebo reference="${prefix}_caster_back_link">
+      <mu1>0.1</mu1>
+      <mu2>0.1</mu2>
+      <kp>1000000.0</kp>
+      <kd>100.0</kd>
+      <minDepth>0.001</minDepth>
+      <maxVel>1.0</maxVel>
+      <material>Gazebo/FlatBlack</material>
+	</gazebo>
+	<gazebo reference="${prefix}_imu_link">
+      <sensor type="imu" name="imu">
+		<always_on>true</always_on>
+		<visualize>$(arg imu_visual)</visualize>
+      </sensor>
+      <material>Gazebo/FlatBlack</material>
+	</gazebo>
+	<gazebo>
+      <plugin name="turtlebot3_burger_controller" filename="libgazebo_ros_diff_drive.so">
+		<commandTopic>${prefix}/cmd_vel</commandTopic>
+		<odometryTopic>${prefix}/odom</odometryTopic>
+		<odometryFrame>${prefix}/odom</odometryFrame>
+		<odometrySource>world</odometrySource>
+		<publishOdomTF>true</publishOdomTF>
+		<robotBaseFrame>${prefix}_base_footprint</robotBaseFrame>
+		<publishWheelTF>false</publishWheelTF>
+		<publishTf>true</publishTf>
+		<publishWheelJointState>true</publishWheelJointState>
+		<legacyMode>false</legacyMode>
+		<updateRate>30</updateRate>
+		<leftJoint>${prefix}_wheel_left_joint</leftJoint>
+		<rightJoint>${prefix}_wheel_right_joint</rightJoint>
+		<wheelSeparation>0.160</wheelSeparation>
+		<wheelDiameter>0.066</wheelDiameter>
+		<wheelAcceleration>1</wheelAcceleration>
+		<wheelTorque>10</wheelTorque>
+		<rosDebugLevel>na</rosDebugLevel>
       </plugin>
-    </sensor>
-  </gazebo>
+	</gazebo>
+	<gazebo>
+      <plugin name="imu_plugin" filename="libgazebo_ros_imu.so">
+		<alwaysOn>true</alwaysOn>
+		<bodyName>${prefix}_imu_link</bodyName>
+		<frameName>${prefix}_imu_link</frameName>
+		<topicName>${prefix}/imu</topicName>
+		<serviceName>${prefix}/imu_service</serviceName>
+		<gaussianNoise>0.0</gaussianNoise>
+		<updateRate>0</updateRate>
+		<imu>
+          <noise>
+			<type>gaussian</type>
+			<rate>
+              <mean>0.0</mean>
+              <stddev>2e-4</stddev>
+              <bias_mean>0.0000075</bias_mean>
+              <bias_stddev>0.0000008</bias_stddev>
+			</rate>
+			<accel>
+              <mean>0.0</mean>
+              <stddev>1.7e-2</stddev>
+              <bias_mean>0.1</bias_mean>
+              <bias_stddev>0.001</bias_stddev>
+			</accel>
+          </noise>
+		</imu>
+      </plugin>
+	</gazebo>
+	<gazebo reference="${prefix}_base_scan">
+      <material>Gazebo/FlatBlack</material>
+      <sensor type="ray" name="lds_lfcd_sensor">
+		<pose>0 0 0 0 0 0</pose>
+		<visualize>$(arg laser_visual)</visualize>
+		<update_rate>5</update_rate>
+		<ray>
+          <scan>
+			<horizontal>
+              <samples>360</samples>
+              <resolution>1</resolution>
+              <min_angle>0.0</min_angle>
+              <max_angle>6.28319</max_angle>
+			</horizontal>
+          </scan>
+          <range>
+			<min>0.120</min>
+			<max>3.5</max>
+			<resolution>0.015</resolution>
+          </range>
+          <noise>
+			<type>gaussian</type>
+			<mean>0.0</mean>
+			<stddev>0.01</stddev>
+          </noise>
+		</ray>
+		<plugin name="gazebo_ros_lds_lfcd_controller" filename="libgazebo_ros_laser.so">
+          <topicName>${prefix}/scan</topicName>
+          <frameName>${prefix}_base_scan</frameName>
+		</plugin>
+      </sensor>
+	</gazebo>
+  </xacro:macro>
 </robot>

File: turtlebot3_custom_description/urdf/turtlebot3_burger.urdf.xacro (robot description, xacro)
@@ -1,17 +1,19 @@
 <?xml version="1.0" ?>
 <robot name="turtlebot3_burger" xmlns:xacro="http://ros.org/wiki/xacro">
-  <xacro:include filename="$(find turtlebot3_description)/urdf/common_properties.xacro"/>
-  <xacro:include filename="$(find turtlebot3_description)/urdf/turtlebot3_burger.gazebo.xacro"/>
-  <link name="base_footprint"/>
-  <joint name="base_joint" type="fixed">
-    <parent link="base_footprint"/>
-    <child link="base_link"/>
+  <xacro:arg name="robot_namespace" default="burger1"/>
+  <xacro:include filename="$(find turtlebot3_custom_description)/urdf/common_properties.xacro"/>
+  <xacro:include filename="$(find turtlebot3_custom_description)/urdf/turtlebot3_burger.gazebo.xacro"/>
+  <burger_sensor_macro prefix="burger1"/>
+  <link name="$(arg robot_namespace)_base_footprint"/>
+  <joint name="$(arg robot_namespace)_base_joint" type="fixed">
+    <parent link="$(arg robot_namespace)_base_footprint"/>
+    <child link="$(arg robot_namespace)_base_link"/>
     <origin xyz="0.0 0.0 0.010" rpy="0 0 0"/>
   </joint>
-  <link name="base_link">
+  <link name="$(arg robot_namespace)_base_link">
     <visual>
       <origin xyz="-0.032 0 0.0" rpy="0 0 0"/>
       <geometry>
-        <mesh filename="package://turtlebot3_description/meshes/bases/burger_base.stl" scale="0.001 0.001 0.001"/>
+        <mesh filename="package://turtlebot3_custom_description/meshes/bases/burger_base.stl" scale="0.001 0.001 0.001"/>
       </geometry>
       <material name="light_black"/>
@@ -31,15 +33,15 @@
     </inertial>
   </link>
-  <joint name="wheel_left_joint" type="continuous">
-    <parent link="base_link"/>
-    <child link="wheel_left_link"/>
+  <joint name="$(arg robot_namespace)_wheel_left_joint" type="continuous">
+    <parent link="$(arg robot_namespace)_base_link"/>
+    <child link="$(arg robot_namespace)_wheel_left_link"/>
     <origin xyz="0.0 0.08 0.023" rpy="-1.57 0 0"/>
     <axis xyz="0 0 1"/>
   </joint>
-  <link name="wheel_left_link">
+  <link name="$(arg robot_namespace)_wheel_left_link">
     <visual>
       <origin xyz="0 0 0" rpy="1.57 0 0"/>
       <geometry>
-        <mesh filename="package://turtlebot3_description/meshes/wheels/left_tire.stl" scale="0.001 0.001 0.001"/>
+        <mesh filename="package://turtlebot3_custom_description/meshes/wheels/left_tire.stl" scale="0.001 0.001 0.001"/>
       </geometry>
       <material name="dark"/>
@@ -59,15 +61,15 @@
       </inertial>
   </link>
-  <joint name="wheel_right_joint" type="continuous">
-    <parent link="base_link"/>
-    <child link="wheel_right_link"/>
+  <joint name="$(arg robot_namespace)_wheel_right_joint" type="continuous">
+    <parent link="$(arg robot_namespace)_base_link"/>
+    <child link="$(arg robot_namespace)_wheel_right_link"/>
     <origin xyz="0.0 -0.080 0.023" rpy="-1.57 0 0"/>
     <axis xyz="0 0 1"/>
   </joint>
-  <link name="wheel_right_link">
+  <link name="$(arg robot_namespace)_wheel_right_link">
     <visual>
       <origin xyz="0 0 0" rpy="1.57 0 0"/>
       <geometry>
-        <mesh filename="package://turtlebot3_description/meshes/wheels/right_tire.stl" scale="0.001 0.001 0.001"/>
+        <mesh filename="package://turtlebot3_custom_description/meshes/wheels/right_tire.stl" scale="0.001 0.001 0.001"/>
       </geometry>
       <material name="dark"/>
@@ -87,10 +89,10 @@
       </inertial>
   </link>
-  <joint name="caster_back_joint" type="fixed">
-    <parent link="base_link"/>
-    <child link="caster_back_link"/>
+  <joint name="$(arg robot_namespace)_caster_back_joint" type="fixed">
+    <parent link="$(arg robot_namespace)_base_link"/>
+    <child link="$(arg robot_namespace)_caster_back_link"/>
     <origin xyz="-0.081 0 -0.004" rpy="-1.57 0 0"/>
   </joint>
-  <link name="caster_back_link">
+  <link name="$(arg robot_namespace)_caster_back_link">
     <collision>
       <origin xyz="0 0.001 0" rpy="0 0 0"/>
@@ -107,20 +109,20 @@
     </inertial>
   </link>
-  <joint name="imu_joint" type="fixed">
-    <parent link="base_link"/>
-    <child link="imu_link"/>
+  <joint name="$(arg robot_namespace)_imu_joint" type="fixed">
+    <parent link="$(arg robot_namespace)_base_link"/>
+    <child link="$(arg robot_namespace)_imu_link"/>
     <origin xyz="-0.032 0 0.068" rpy="0 0 0"/>
   </joint>
-  <link name="imu_link"/>
-  <joint name="scan_joint" type="fixed">
-    <parent link="base_link"/>
-    <child link="base_scan"/>
+  <link name="$(arg robot_namespace)_imu_link"/>
+  <joint name="$(arg robot_namespace)_scan_joint" type="fixed">
+    <parent link="$(arg robot_namespace)_base_link"/>
+    <child link="$(arg robot_namespace)_base_scan"/>
     <origin xyz="-0.032 0 0.172" rpy="0 0 0"/>
   </joint>
-  <link name="base_scan">
+  <link name="$(arg robot_namespace)_base_scan">
     <visual>
       <origin xyz="0 0 0.0" rpy="0 0 0"/>
       <geometry>
-        <mesh filename="package://turtlebot3_description/meshes/sensors/lds.stl" scale="0.001 0.001 0.001"/>
+        <mesh filename="package://turtlebot3_custom_description/meshes/sensors/lds.stl" scale="0.001 0.001 0.001"/>
       </geometry>
       <material name="dark"/>

Commit message: also works with waffle
Signed-off-by: soblin <hilo.soblin@gmail.com>

File: turtlebot3_custom_description/urdf/turtlebot3_burger.gazebo.xacro (robot description, xacro)
@@ -95,5 +95,6 @@
       <sensor type="ray" name="lds_lfcd_sensor">
         <always_on>true</always_on>
-        <visualize>true</visualize>
+		<!-- if true you can see the ray on gazebo -->
+		<visualize>$(arg laser_visual)</visualize>
         <pose>-0.032 0 0.171 0 0 0</pose>
         <update_rate>5</update_rate>

File: turtlebot3_custom_description/urdf/turtlebot3_waffle.gazebo.xacro (robot description, xacro)
@@ -55,26 +55,25 @@
 	<gazebo>
       <plugin name="turtlebot3_waffle_controller" filename="libgazebo_ros_diff_drive.so">
-		<commandTopic>${prefix}_cmd_vel</commandTopic>
-		<odometryTopic>${prefix}_odom</odometryTopic>
-		<odometryFrame>${prefix}_odom</odometryFrame>
-		<odometrySource>world</odometrySource>
-		<publishOdomTF>true</publishOdomTF>
-		<robotBaseFrame>${prefix}_base_footprint</robotBaseFrame>
-		<publishWheelTF>false</publishWheelTF>
-		<publishTf>true</publishTf>
-		<publishWheelJointState>true</publishWheelJointState>
-		<legacyMode>false</legacyMode>
-		<updateRate>30</updateRate>
-		<leftJoint>${prefix}_wheel_left_joint</leftJoint>
-		<rightJoint>${prefix}_wheel_right_joint</rightJoint>
-		<wheelSeparation>0.287</wheelSeparation>
-		<wheelDiameter>0.066</wheelDiameter>
-		<wheelAcceleration>1</wheelAcceleration>
-		<wheelTorque>10</wheelTorque>
-		<rosDebugLevel>na</rosDebugLevel>
+		<update_rate>30</update_rate>
+		<left_joint>${prefix}_wheel_left_joint</left_joint>
+		<right_joint>${prefix}_wheel_right_joint</right_joint>
+		<wheel_separation>0.287</wheel_separation>
+		<wheel_diameter>0.066</wheel_diameter>
+		<max_wheel_acceleration>1</max_wheel_acceleration>
+		<max_wheel_torque>10</max_wheel_torque>
+		<publish_odom>true</publish_odom>
+		<publish_odom_tf>true</publish_odom_tf>
+		<publish_wheel_tf>false</publish_wheel_tf>
+		<odometry_frame>${prefix}_odom</odometry_frame>
+		<robot_base_frame>${prefix}_base_footprint</robot_base_frame>
+		<!-- https://github.com/ros-simulation/gazebo_ros_pkgs/wiki/ROS-2-Migration:-Diff-drive -->
+		<ros>
+		  <remapping>cmd_vel:=${prefix}_cmd_vel</remapping>
+		  <remapping>odom:=${prefix}_odom</remapping>
+		</ros>
       </plugin>
 	</gazebo>
-	<gazebo>
-      <plugin name="imu_plugin" filename="libgazebo_ros_imu.so">
+	<!--gazebo>
+		<plugin name="imu_plugin" filename="libgazebo_ros_imu.so">
 		<alwaysOn>true</alwaysOn>
 		<bodyName>${prefix}_imu_link</bodyName>
@@ -85,26 +84,27 @@
 		<updateRate>0</updateRate>
 		<imu>
-          <noise>
-			<type>gaussian</type>
-			<rate>
-              <mean>0.0</mean>
-              <stddev>2e-4</stddev>
-              <bias_mean>0.0000075</bias_mean>
-              <bias_stddev>0.0000008</bias_stddev>
-			</rate>
-			<accel>
-              <mean>0.0</mean>
-              <stddev>1.7e-2</stddev>
-              <bias_mean>0.1</bias_mean>
-              <bias_stddev>0.001</bias_stddev>
-			</accel>
-          </noise>
+        <noise>
+		<type>gaussian</type>
+		<rate>
+        <mean>0.0</mean>
+        <stddev>2e-4</stddev>
+        <bias_mean>0.0000075</bias_mean>
+        <bias_stddev>0.0000008</bias_stddev>
+		</rate>
+		<accel>
+        <mean>0.0</mean>
+        <stddev>1.7e-2</stddev>
+        <bias_mean>0.1</bias_mean>
+        <bias_stddev>0.001</bias_stddev>
+		</accel>
+        </noise>
 		</imu>
-      </plugin>
-	</gazebo>
+		</plugin>
+		</gazebo-->
 	<gazebo reference="${prefix}_base_scan">
-      <material>Gazebo/FlatBlack</material>
       <sensor type="ray" name="lds_lfcd_sensor">
+        <always_on>true</always_on>
 		<pose>0 0 0 0 0 0</pose>
+		<!-- if true you can see the ray on gazebo -->
 		<visualize>$(arg laser_visual)</visualize>
 		<update_rate>5</update_rate>
@@ -129,7 +129,10 @@
           </noise>
 		</ray>
-		<plugin name="gazebo_ros_lds_lfcd_controller" filename="libgazebo_ros_laser.so">
-          <topicName>${prefix}_scan</topicName>
-          <frameName>${prefix}_base_scan</frameName>
+		<plugin name="gazebo_ros_lds_lfcd_controller" filename="libgazebo_ros_ray_sensor.so">
+          <ros>
+            <remapping>~/out:=${prefix}_scan</remapping>
+          </ros>
+          <output_type>sensor_msgs/LaserScan</output_type>
+          <frame_name>${prefix}_base_scan</frame_name>
 		</plugin>
       </sensor>
@@ -137,8 +140,9 @@
 	<gazebo reference="${prefix}_camera_rgb_frame">
       <sensor type="depth" name="realsense_R200">
-		<always_on>true</always_on>
-		<visualize>$(arg camera_visual)</visualize>
-		<camera>
-          <horizontal_fov>1.3439</horizontal_fov>
+        <always_on>true</always_on>
+        <visualize>true</visualize>
+        <update_rate>30</update_rate>
+        <camera name="intel_realsense_r200">
+          <horizontal_fov>1.02974</horizontal_fov>
           <image>
             <width>1920</width>
@@ -146,34 +150,27 @@
             <format>R8G8B8</format>
           </image>
-          <depth_camera></depth_camera>
           <clip>
-            <near>0.03</near>
-            <far>100</far>
+            <near>0.02</near>
+            <far>300</far>
           </clip>
-		</camera>
-		<plugin name="camera_controller" filename="libgazebo_ros_openni_kinect.so">
-          <baseline>0.2</baseline>
-          <alwaysOn>true</alwaysOn>
-          <updateRate>30.0</updateRate>
-          <cameraName>${prefix}/camera</cameraName>
-          <frameName>${prefix}_camera_rgb_optical_frame</frameName>
-          <imageTopicName>rgb_image_raw</imageTopicName>
-          <depthImageTopicName>depth_image_raw</depthImageTopicName>
-          <pointCloudTopicName>depth_points</pointCloudTopicName>
-          <cameraInfoTopicName>rgb_camera_info</cameraInfoTopicName>
-          <depthImageCameraInfoTopicName>depth_camera_info</depthImageCameraInfoTopicName>
-          <pointCloudCutoff>0.4</pointCloudCutoff>
-          <hackBaseline>0.07</hackBaseline>
-          <distortionK1>0.0</distortionK1>
-          <distortionK2>0.0</distortionK2>
-          <distortionK3>0.0</distortionK3>
-          <distortionT1>0.0</distortionT1>
-          <distortionT2>0.0</distortionT2>
-          <CxPrime>0.0</CxPrime>
-          <Cx>0.0</Cx>
-          <Cy>0.0</Cy>
-          <focalLength>0</focalLength>
-          <hackBaseline>0</hackBaseline>
-		</plugin>
+          <noise>
+            <type>gaussian</type>
+            <!-- Noise is sampled independently per pixel on each frame.
+                 That pixel's noise value is added to each of its color
+                 channels, which at that point lie in the range [0,1]. -->
+            <mean>0.0</mean>
+            <stddev>0.007</stddev>
+          </noise>
+        </camera>
+        <plugin name="camera_driver" filename="libgazebo_ros_camera.so">
+          <ros>
+            <!-- <namespace>test_cam</namespace> -->
+            <!-- <remapping>image_raw:=image_demo</remapping> -->
+            <!-- <remapping>camera_info:=camera_info_demo</remapping> -->
+          </ros>
+          <!-- camera_name>omit so it defaults to sensor name</camera_name-->
+          <!-- frame_name>omit so it defaults to link name</frameName-->
+          <!-- <hack_baseline>0.07</hack_baseline> -->
+        </plugin>
       </sensor>
 	</gazebo>

File: turtlebot3_custom_description/urdf/turtlebot3_waffle.urdf.xacro (robot description, xacro)
@@ -19,5 +19,5 @@
       <origin xyz="-0.064 0 0.0" rpy="0 0 0"/>
       <geometry>
-        <mesh filename="package://turtlebot3_custom_description/meshes/bases/waffle_base.stl" scale="0.001 0.001 0.001"/>
+        <mesh filename="package://turtlebot3_custom_description/meshes/waffle_base.dae" scale="0.001 0.001 0.001"/>
       </geometry>
       <material name="light_black"/>
@@ -47,5 +47,5 @@
       <origin xyz="0 0 0" rpy="1.57 0 0"/>
       <geometry>
-        <mesh filename="package://turtlebot3_custom_description/meshes/wheels/left_tire.stl" scale="0.001 0.001 0.001"/>
+        <mesh filename="package://turtlebot3_custom_description/meshes/tire.dae" scale="0.001 0.001 0.001"/>
       </geometry>
       <material name="dark"/>
@@ -75,5 +75,5 @@
       <origin xyz="0 0 0" rpy="1.57 0 0"/>
       <geometry>
-        <mesh filename="package://turtlebot3_custom_description/meshes/wheels/right_tire.stl" scale="0.001 0.001 0.001"/>
+        <mesh filename="package://turtlebot3_custom_description/meshes/tire.dae" scale="0.001 0.001 0.001"/>
       </geometry>
       <material name="dark"/>
@@ -148,5 +148,5 @@
       <origin xyz="0 0 0" rpy="0 0 0"/>
       <geometry>
-        <mesh filename="package://turtlebot3_custom_description/meshes/sensors/lds.stl" scale="0.001 0.001 0.001"/>
+        <mesh filename="package://turtlebot3_custom_description/meshes/lds.dae" scale="0.001 0.001 0.001"/>
       </geometry>
       <material name="dark"/>
@@ -175,5 +175,5 @@
       <origin xyz="0 0 0" rpy="1.57 0 1.57"/>
       <geometry>
-		<mesh filename="package://turtlebot3_custom_description/meshes/sensors/r200.dae" />
+		<mesh filename="package://turtlebot3_custom_description/meshes/r200.dae" />
       </geometry>
     </visual>
